Commit message: initial coommit

File: bot1/bot1_description_dev/urdf/bot1_description_dev.urdf (robot description, URDF)
Before this commit: robot bot1_description_dev, 9 links, 8 joints
Joints:
- joint whee_bl_joint: type continuous -> fixed
- joint wheel_br_joint: type continuous -> fixed
- joint wheel_fl_joint: type continuous -> fixed
- joint wheel_fr_joint: type continuous -> fixed

Commit message: initial commit

File: bot1/bot1_description_dev/urdf/bot1_description_dev.urdf (robot description, URDF)
Before this commit: robot bot1_description_dev, 9 links, 8 joints
Links:
- added link imu_link, mass 0.0007817846555206; collision mesh filename=package://bot1_description_dev/meshes/imu_link.STL; visual mesh filename=package://bot1_description_dev/meshes/imu_link.STL
- link base_link: mass 15.9642902147073 -> 15.998
- link camera_link: mass 0.0441644560542025 -> 0.0441644560541813
- link kinect_link: mass 0.658662539657532 -> 0.658662539657539
- link wheel_bl_link: mass 0.688491418307573 -> 0.688491418307572
- link wheel_br_link: mass 0.688491418307572 -> 0
- link wheel_fl_link: mass 0.688491418307573 -> 0.688491418307572
Joints:
- removed joint whee_bl_joint
- added joint imu_joint: type fixed, parent base_link, child imu_link, origin xyz=-0.052 0.098 0.168 rpy=1.5708 0 0, axis 0 0 0
- added joint wheel_bl_joint: type fixed, parent base_link, child wheel_bl_link, origin xyz=-0.26302 0.26302 0.0755 rpy=-1.5708 -0.37436 -2.3562, axis 0 0 -1
- joint base_joint: axis (none) -> 0 0 0; origin xyz=0.0 0.0 0.0 rpy=0 0 0 -> xyz=0 0 0 rpy=0 0 0
- joint camera_joint: origin xyz=0.480360774189096 -0.685219620888692 0.812857605494797 rpy=-3.14159265358979 0 3.14159265358979 -> xyz=0.15402 0.0034297 0.45835 rpy=3.1416 0 -1.5708
- joint kinect_joint: origin xyz=0.47693234400763 -0.703241129330077 0.744511564271028 rpy=1.50898907863485 0 0 -> xyz=0.17504 0 0.39 rpy=1.6326 0 1.5708
- joint scan_joint: origin xyz=0.476931055313594 -0.935335323699936 0.424610253244008 rpy=-1.5707963267949 0 -1.5707963267949 -> xyz=0.40414 0 0.0701 rpy=1.5708 0 0
- joint wheel_br_joint: axis 0 0 0 -> 0 0 1; origin xyz=0.213906740303079 -0.268171008689424 0.430010253244007 rpy=-1.57079632679489 -0.374361018706128 -2.35619449019234 -> xyz=-0.26302 -0.26302 0.0755 rpy=-1.5708 -0.37436 -0.7854
- joint wheel_fl_joint: axis 0 0 0 -> 0 0 -1; origin xyz=0.739955370324104 -0.794219638710453 0.430010253244007 rpy=-1.5707963267949 -0.374361018706124 0.785398163397448 -> xyz=0.26302 0.26302 0.0755 rpy=-1.5708 -0.37436 2.3562
- joint wheel_fr_joint: axis 0 0 0 -> 0 0 -1; origin xyz=0.213906740303084 -0.794219638710449 0.430010253244008 rpy=-1.5707963267949 -0.374361018706124 -0.785398163397452 -> xyz=0.26302 -0.26302 0.0755 rpy=-1.5708 -0.37436 0.7854

Commit message: initial commit

File: bot1/bot1_description_dev/urdf/bot1_description_dev.urdf (robot description, URDF)
Before this commit: robot bot1_description_dev, 10 links, 9 joints
Joints:
- joint scan_joint: origin xyz=0.40414 0 0.0701 rpy=1.5708 0 0 -> xyz=0.40414 0 0.0701 rpy=0 0 0
